Commit message: Changes to facilitate transition from fmauch_universal_robots
Make kinematic planning config match.
Load joint limits using the *_joint suffix on all joints.
Use the base_link correction instead of the base_link_inertia frame.
Remove flange and tool0 links + associated joints.
Add gazebo self-collision definition.

File: ur_description/urdf/inc/ur_common.xacro (robot description, xacro)
@@ -37,28 +37,28 @@
     <xacro:property name="sec_kinematics" value="${config_kinematics_parameters['kinematics']}" />
     <!-- JOINTS LIMIT PARAMETERS -->
-    <xacro:property name="shoulder_pan_lower_limit" value="${sec_limits['shoulder_pan']['min_position']}" scope="parent"/>
-    <xacro:property name="shoulder_pan_upper_limit" value="${sec_limits['shoulder_pan']['max_position']}" scope="parent"/>
-    <xacro:property name="shoulder_pan_velocity_limit" value="${sec_limits['shoulder_pan']['max_velocity']}" scope="parent"/>
-    <xacro:property name="shoulder_pan_effort_limit" value="${sec_limits['shoulder_pan']['max_effort']}" scope="parent"/>
-    <xacro:property name="shoulder_lift_lower_limit" value="${sec_limits['shoulder_lift']['min_position']}" scope="parent"/>
-    <xacro:property name="shoulder_lift_upper_limit" value="${sec_limits['shoulder_lift']['max_position']}" scope="parent"/>
-    <xacro:property name="shoulder_lift_velocity_limit" value="${sec_limits['shoulder_lift']['max_velocity']}" scope="parent"/>
-    <xacro:property name="shoulder_lift_effort_limit" value="${sec_limits['shoulder_lift']['max_effort']}" scope="parent"/>
+    <xacro:property name="shoulder_pan_lower_limit" value="${sec_limits['shoulder_pan_joint']['min_position']}" scope="parent"/>
+    <xacro:property name="shoulder_pan_upper_limit" value="${sec_limits['shoulder_pan_joint']['max_position']}" scope="parent"/>
+    <xacro:property name="shoulder_pan_velocity_limit" value="${sec_limits['shoulder_pan_joint']['max_velocity']}" scope="parent"/>
+    <xacro:property name="shoulder_pan_effort_limit" value="${sec_limits['shoulder_pan_joint']['max_effort']}" scope="parent"/>
+    <xacro:property name="shoulder_lift_lower_limit" value="${sec_limits['shoulder_lift_joint']['min_position']}" scope="parent"/>
+    <xacro:property name="shoulder_lift_upper_limit" value="${sec_limits['shoulder_lift_joint']['max_position']}" scope="parent"/>
+    <xacro:property name="shoulder_lift_velocity_limit" value="${sec_limits['shoulder_lift_joint']['max_velocity']}" scope="parent"/>
+    <xacro:property name="shoulder_lift_effort_limit" value="${sec_limits['shoulder_lift_joint']['max_effort']}" scope="parent"/>
     <xacro:property name="elbow_joint_lower_limit" value="${sec_limits['elbow_joint']['min_position']}" scope="parent"/>
     <xacro:property name="elbow_joint_upper_limit" value="${sec_limits['elbow_joint']['max_position']}" scope="parent"/>
     <xacro:property name="elbow_joint_velocity_limit" value="${sec_limits['elbow_joint']['max_velocity']}" scope="parent"/>
     <xacro:property name="elbow_joint_effort_limit" value="${sec_limits['elbow_joint']['max_effort']}" scope="parent"/>
-    <xacro:property name="wrist_1_lower_limit" value="${sec_limits['wrist_1']['min_position']}" scope="parent"/>
-    <xacro:property name="wrist_1_upper_limit" value="${sec_limits['wrist_1']['max_position']}" scope="parent"/>
-    <xacro:property name="wrist_1_velocity_limit" value="${sec_limits['wrist_1']['max_velocity']}" scope="parent"/>
-    <xacro:property name="wrist_1_effort_limit" value="${sec_limits['wrist_1']['max_effort']}" scope="parent"/>
-    <xacro:property name="wrist_2_lower_limit" value="${sec_limits['wrist_2']['min_position']}" scope="parent"/>
-    <xacro:property name="wrist_2_upper_limit" value="${sec_limits['wrist_2']['max_position']}" scope="parent"/>
-    <xacro:property name="wrist_2_velocity_limit" value="${sec_limits['wrist_2']['max_velocity']}" scope="parent"/>
-    <xacro:property name="wrist_2_effort_limit" value="${sec_limits['wrist_2']['max_effort']}" scope="parent"/>
-    <xacro:property name="wrist_3_lower_limit" value="${sec_limits['wrist_3']['min_position']}" scope="parent"/>
-    <xacro:property name="wrist_3_upper_limit" value="${sec_limits['wrist_3']['max_position']}" scope="parent"/>
-    <xacro:property name="wrist_3_velocity_limit" value="${sec_limits['wrist_3']['max_velocity']}" scope="parent"/>
-    <xacro:property name="wrist_3_effort_limit" value="${sec_limits['wrist_3']['max_effort']}" scope="parent"/>
+    <xacro:property name="wrist_1_lower_limit" value="${sec_limits['wrist_1_joint']['min_position']}" scope="parent"/>
+    <xacro:property name="wrist_1_upper_limit" value="${sec_limits['wrist_1_joint']['max_position']}" scope="parent"/>
+    <xacro:property name="wrist_1_velocity_limit" value="${sec_limits['wrist_1_joint']['max_velocity']}" scope="parent"/>
+    <xacro:property name="wrist_1_effort_limit" value="${sec_limits['wrist_1_joint']['max_effort']}" scope="parent"/>
+    <xacro:property name="wrist_2_lower_limit" value="${sec_limits['wrist_2_joint']['min_position']}" scope="parent"/>
+    <xacro:property name="wrist_2_upper_limit" value="${sec_limits['wrist_2_joint']['max_position']}" scope="parent"/>
+    <xacro:property name="wrist_2_velocity_limit" value="${sec_limits['wrist_2_joint']['max_velocity']}" scope="parent"/>
+    <xacro:property name="wrist_2_effort_limit" value="${sec_limits['wrist_2_joint']['max_effort']}" scope="parent"/>
+    <xacro:property name="wrist_3_lower_limit" value="${sec_limits['wrist_3_joint']['min_position']}" scope="parent"/>
+    <xacro:property name="wrist_3_upper_limit" value="${sec_limits['wrist_3_joint']['max_position']}" scope="parent"/>
+    <xacro:property name="wrist_3_velocity_limit" value="${sec_limits['wrist_3_joint']['max_velocity']}" scope="parent"/>
+    <xacro:property name="wrist_3_effort_limit" value="${sec_limits['wrist_3_joint']['max_effort']}" scope="parent"/>
     <!-- kinematics -->
     <xacro:property name="shoulder_x" value="${sec_kinematics['shoulder']['x']}" scope="parent"/>

File: ur_description/urdf/inc/ur_macro.xacro (robot description, xacro)
@@ -63,9 +63,14 @@
     <!-- Add URDF transmission elements (for ros_control) -->
     <xacro:ur_arm_transmission prefix="${prefix}" hw_interface="${transmission_hw_interface}" />
+    <!--
+      This is for compatibility reasons, as transformation between base and
+      base_link was always 180 degree in the ur_description.
+    -->
+    <!-- TODO(cj): See if we can remove this in favor of the new base_link_inertia link. -->
+    <xacro:property name="base_correction" value="${pi}" />
     <!-- links: main serial chain -->
-    <link name="${prefix}base_link"/>
-    <link name="${prefix}base_link_inertia">
-      <visual>
-        <origin xyz="0 0 0" rpy="0 0 ${pi}"/>
+    <link name="${prefix}base_link">
+      <visual>
+        <origin xyz="0 0 0" rpy="0 0 ${base_correction}"/>
         <geometry>
           <mesh filename="${base_visual_mesh}"/>
@@ -76,5 +81,5 @@
       </visual>
       <collision>
-        <origin xyz="0 0 0" rpy="0 0 ${pi}"/>
+        <origin xyz="0 0 0" rpy="0 0 ${base_correction}"/>
         <geometry>
           <mesh filename="${base_collision_mesh}"/>
@@ -265,18 +270,8 @@
     </link>
     <!-- joints: main serial chain -->
-    <joint name="${prefix}base_link-base_link_inertia" type="fixed">
+    <joint name="${prefix}shoulder_pan_joint" type="revolute">
       <parent link="${prefix}base_link" />
-      <child link="${prefix}base_link_inertia" />
-      <!-- 'base_link' is REP-103 aligned (so X+ forward), while the internal
-           frames of the robot/controller have X+ pointing backwards.
-           Use the joint between 'base_link' and 'base_link_inertia' (a dummy
-           link/frame) to introduce the necessary rotation over Z (of pi rad).
-      -->
-      <origin xyz="0 0 0" rpy="0 0 ${pi}" />
-    </joint>
-    <joint name="${prefix}shoulder_pan_joint" type="revolute">
-      <parent link="${prefix}base_link_inertia" />
       <child link="${prefix}shoulder_link" />
-      <origin xyz="${shoulder_x} ${shoulder_y} ${shoulder_z}" rpy="${shoulder_roll} ${shoulder_pitch} ${shoulder_yaw}" />
+      <origin xyz="${shoulder_x} ${shoulder_y} ${shoulder_z}" rpy="${shoulder_roll} ${shoulder_pitch} ${shoulder_yaw - base_correction}" />
       <axis xyz="0 0 1" />
       <limit lower="${shoulder_pan_lower_limit}" upper="${shoulder_pan_upper_limit}"
@@ -355,23 +350,35 @@
            the UR controller.
       -->
-      <origin xyz="0 0 0" rpy="0 0 ${pi}"/>
+      <origin xyz="0 0 0" rpy="0 0 ${base_correction}"/>
       <parent link="${prefix}base_link"/>
       <child link="${prefix}base"/>
     </joint>
-    <!-- ROS-Industrial 'flange' frame: attachment point for EEF models -->
-    <link name="${prefix}flange" />
-    <joint name="${prefix}wrist_3-flange" type="fixed">
-      <parent link="${prefix}wrist_3_link" />
-      <child link="${prefix}flange" />
-      <origin xyz="0 0 0" rpy="0 ${-pi/2.0} ${-pi/2.0}" />
-    </joint>
-    <!-- ROS-Industrial 'tool0' frame: all-zeros tool frame -->
-    <link name="${prefix}tool0"/>
-    <joint name="${prefix}flange-tool0" type="fixed">
-      <!-- default toolframe: X+ left, Y+ up, Z+ front -->
-      <origin xyz="0 0 0" rpy="${pi/2.0} 0 ${pi/2.0}"/>
-      <parent link="${prefix}flange"/>
-      <child link="${prefix}tool0"/>
-    </joint>
+    <!--
+      TODO(cj): See if we can keep the flange and tool0 links and their
+        corresponding joints.
+    -->
+    <!-- Configure self collision properties per link -->
+    <!-- TODO(cj): Have callers use the ur_robot_gazebo macro instead. -->
+    <gazebo reference="${prefix}shoulder_link">
+      <selfCollide>true</selfCollide>
+    </gazebo>
+    <gazebo reference="${prefix}upper_arm_link">
+      <selfCollide>true</selfCollide>
+    </gazebo>
+    <gazebo reference="${prefix}forearm_link">
+      <selfCollide>true</selfCollide>
+    </gazebo>
+    <gazebo reference="${prefix}wrist_1_link">
+      <selfCollide>true</selfCollide>
+    </gazebo>
+    <gazebo reference="${prefix}wrist_3_link">
+      <selfCollide>true</selfCollide>
+    </gazebo>
+    <gazebo reference="${prefix}wrist_2_link">
+      <selfCollide>true</selfCollide>
+    </gazebo>
+    <gazebo reference="${prefix}ee_link">
+      <selfCollide>true</selfCollide>
+    </gazebo>
   </xacro:macro>
 </robot>

Commit message: Add `motor_dynamics` processing
Also define motor dynamics for UR5e

File: ur_description/urdf/inc/ur_common.xacro (robot description, xacro)
@@ -34,4 +34,5 @@
     <xacro:property name="sec_offsets" value="${config_physical_parameters['offsets']}"/>
     <xacro:property name="sec_inertia_parameters" value="${config_physical_parameters['inertia_parameters']}" />
+    <xacro:property name="sec_motor_dynamics" value="${config_physical_parameters['motor_dynamics']}" />
     <xacro:property name="sec_mesh_files" value="${config_visual_parameters['mesh_files']}" />
     <xacro:property name="sec_kinematics" value="${config_kinematics_parameters['kinematics']}" />
@@ -61,4 +62,35 @@
     <xacro:property name="wrist_3_velocity_limit" value="${sec_limits['wrist_3_joint']['max_velocity']}" scope="parent"/>
     <xacro:property name="wrist_3_effort_limit" value="${sec_limits['wrist_3_joint']['max_effort']}" scope="parent"/>
+    <!-- MOTOR DYNAMICS PARAMETERS -->
+    <xacro:property name="shoulder_pan_joint_static_friction" value="${sec_motor_dynamics['shoulder_pan_joint']['static_friction']}" scope="parent"/>
+    <xacro:property name="shoulder_pan_joint_viscous_friction" value="${sec_motor_dynamics['shoulder_pan_joint']['viscous_friction']}" scope="parent"/>
+    <xacro:property name="shoulder_pan_joint_gear_ratio" value="${sec_motor_dynamics['shoulder_pan_joint']['gear_ratio']}" scope="parent"/>
+    <xacro:property name="shoulder_pan_joint_rotor_inertia" value="${sec_motor_dynamics['shoulder_pan_joint']['rotor_inertia']}" scope="parent"/>
+    <xacro:property name="shoulder_pan_joint_reducer_inertia" value="${sec_motor_dynamics['shoulder_pan_joint']['reducer_inertia']}" scope="parent"/>
+    <xacro:property name="shoulder_lift_joint_static_friction" value="${sec_motor_dynamics['shoulder_lift_joint']['static_friction']}" scope="parent"/>
+    <xacro:property name="shoulder_lift_joint_viscous_friction" value="${sec_motor_dynamics['shoulder_lift_joint']['viscous_friction']}" scope="parent"/>
+    <xacro:property name="shoulder_lift_joint_gear_ratio" value="${sec_motor_dynamics['shoulder_lift_joint']['gear_ratio']}" scope="parent"/>
+    <xacro:property name="shoulder_lift_joint_rotor_inertia" value="${sec_motor_dynamics['shoulder_lift_joint']['rotor_inertia']}" scope="parent"/>
+    <xacro:property name="shoulder_lift_joint_reducer_inertia" value="${sec_motor_dynamics['shoulder_lift_joint']['reducer_inertia']}" scope="parent"/>
+    <xacro:property name="elbow_joint_static_friction" value="${sec_motor_dynamics['elbow_joint']['static_friction']}" scope="parent"/>
+    <xacro:property name="elbow_joint_viscous_friction" value="${sec_motor_dynamics['elbow_joint']['viscous_friction']}" scope="parent"/>
+    <xacro:property name="elbow_joint_gear_ratio" value="${sec_motor_dynamics['elbow_joint']['gear_ratio']}" scope="parent"/>
+    <xacro:property name="elbow_joint_rotor_inertia" value="${sec_motor_dynamics['elbow_joint']['rotor_inertia']}" scope="parent"/>
+    <xacro:property name="elbow_joint_reducer_inertia" value="${sec_motor_dynamics['elbow_joint']['reducer_inertia']}" scope="parent"/>
+    <xacro:property name="wrist_1_joint_static_friction" value="${sec_motor_dynamics['wrist_1_joint']['static_friction']}" scope="parent"/>
+    <xacro:property name="wrist_1_joint_viscous_friction" value="${sec_motor_dynamics['wrist_1_joint']['viscous_friction']}" scope="parent"/>
+    <xacro:property name="wrist_1_joint_gear_ratio" value="${sec_motor_dynamics['wrist_1_joint']['gear_ratio']}" scope="parent"/>
+    <xacro:property name="wrist_1_joint_rotor_inertia" value="${sec_motor_dynamics['wrist_1_joint']['rotor_inertia']}" scope="parent"/>
+    <xacro:property name="wrist_1_joint_reducer_inertia" value="${sec_motor_dynamics['wrist_1_joint']['reducer_inertia']}" scope="parent"/>
+    <xacro:property name="wrist_2_joint_static_friction" value="${sec_motor_dynamics['wrist_2_joint']['static_friction']}" scope="parent"/>
+    <xacro:property name="wrist_2_joint_viscous_friction" value="${sec_motor_dynamics['wrist_2_joint']['viscous_friction']}" scope="parent"/>
+    <xacro:property name="wrist_2_joint_gear_ratio" value="${sec_motor_dynamics['wrist_2_joint']['gear_ratio']}" scope="parent"/>
+    <xacro:property name="wrist_2_joint_rotor_inertia" value="${sec_motor_dynamics['wrist_2_joint']['rotor_inertia']}" scope="parent"/>
+    <xacro:property name="wrist_2_joint_reducer_inertia" value="${sec_motor_dynamics['wrist_2_joint']['reducer_inertia']}" scope="parent"/>
+    <xacro:property name="wrist_3_joint_static_friction" value="${sec_motor_dynamics['wrist_3_joint']['static_friction']}" scope="parent"/>
+    <xacro:property name="wrist_3_joint_viscous_friction" value="${sec_motor_dynamics['wrist_3_joint']['viscous_friction']}" scope="parent"/>
+    <xacro:property name="wrist_3_joint_gear_ratio" value="${sec_motor_dynamics['wrist_3_joint']['gear_ratio']}" scope="parent"/>
+    <xacro:property name="wrist_3_joint_rotor_inertia" value="${sec_motor_dynamics['wrist_3_joint']['rotor_inertia']}" scope="parent"/>
+    <xacro:property name="wrist_3_joint_reducer_inertia" value="${sec_motor_dynamics['wrist_3_joint']['reducer_inertia']}" scope="parent"/>
     <!-- kinematics -->
     <xacro:property name="shoulder_x" value="${sec_kinematics['shoulder']['x']}" scope="parent"/>

File: ur_description/urdf/inc/ur_macro.xacro (robot description, xacro)
@@ -281,4 +281,9 @@
       </xacro:if>
       <dynamics damping="0" friction="0"/>
+      <motor_dynamics static_friction="${shoulder_pan_joint_static_friction}"
+                      viscous_friction="${shoulder_pan_joint_viscous_friction}"
+                      gear_ratio="${shoulder_pan_joint_gear_ratio}"
+                      rotor_inertia="${shoulder_pan_joint_rotor_inertia}"
+                      reducer_inertia="${shoulder_pan_joint_reducer_inertia}"/>
     </joint>
     <joint name="${prefix}shoulder_lift_joint" type="revolute">
@@ -293,4 +298,9 @@
       </xacro:if>
       <dynamics damping="0" friction="0"/>
+      <motor_dynamics static_friction="${shoulder_lift_joint_static_friction}"
+                      viscous_friction="${shoulder_lift_joint_viscous_friction}"
+                      gear_ratio="${shoulder_lift_joint_gear_ratio}"
+                      rotor_inertia="${shoulder_lift_joint_rotor_inertia}"
+                      reducer_inertia="${shoulder_lift_joint_reducer_inertia}"/>
     </joint>
     <joint name="${prefix}elbow_joint" type="revolute">
@@ -305,4 +315,9 @@
       </xacro:if>
       <dynamics damping="0" friction="0"/>
+      <motor_dynamics static_friction="${elbow_joint_static_friction}"
+                      viscous_friction="${elbow_joint_viscous_friction}"
+                      gear_ratio="${elbow_joint_gear_ratio}"
+                      rotor_inertia="${elbow_joint_rotor_inertia}"
+                      reducer_inertia="${elbow_joint_reducer_inertia}"/>
     </joint>
     <joint name="${prefix}wrist_1_joint" type="revolute">
@@ -317,4 +332,9 @@
       </xacro:if>
       <dynamics damping="0" friction="0"/>
+      <motor_dynamics static_friction="${wrist_1_joint_static_friction}"
+                      viscous_friction="${wrist_1_joint_viscous_friction}"
+                      gear_ratio="${wrist_1_joint_gear_ratio}"
+                      rotor_inertia="${wrist_1_joint_rotor_inertia}"
+                      reducer_inertia="${wrist_1_joint_reducer_inertia}"/>
     </joint>
     <joint name="${prefix}wrist_2_joint" type="revolute">
@@ -329,4 +349,9 @@
       </xacro:if>
       <dynamics damping="0" friction="0"/>
+      <motor_dynamics static_friction="${wrist_2_joint_static_friction}"
+                      viscous_friction="${wrist_2_joint_viscous_friction}"
+                      gear_ratio="${wrist_2_joint_gear_ratio}"
+                      rotor_inertia="${wrist_2_joint_rotor_inertia}"
+                      reducer_inertia="${wrist_2_joint_reducer_inertia}"/>
     </joint>
     <joint name="${prefix}wrist_3_joint" type="revolute">
@@ -341,4 +366,9 @@
       </xacro:if>
       <dynamics damping="0" friction="0"/>
+      <motor_dynamics static_friction="${wrist_3_joint_static_friction}"
+                      viscous_friction="${wrist_3_joint_viscous_friction}"
+                      gear_ratio="${wrist_3_joint_gear_ratio}"
+                      rotor_inertia="${wrist_3_joint_rotor_inertia}"
+                      reducer_inertia="${wrist_3_joint_reducer_inertia}"/>
     </joint>
     <!-- ROS-Industrial 'base' frame: base_link to UR 'Base' Coordinates transform -->
