Commit message: Rename `motor_dynamics`->`chef_dynamics` + param renaming
`static_friction`->`coulomb_friction`
`viscous_friction`->`viscous_damping`

File: ur_description/urdf/inc/ur_common.xacro (robot description, xacro)
@@ -34,5 +34,5 @@
     <xacro:property name="sec_offsets" value="${config_physical_parameters['offsets']}"/>
     <xacro:property name="sec_inertia_parameters" value="${config_physical_parameters['inertia_parameters']}" />
-    <xacro:property name="sec_motor_dynamics" value="${config_physical_parameters['motor_dynamics']}" />
+    <xacro:property name="sec_joint_dynamics" value="${config_physical_parameters['joint_dynamics']}" />
     <xacro:property name="sec_mesh_files" value="${config_visual_parameters['mesh_files']}" />
     <xacro:property name="sec_kinematics" value="${config_kinematics_parameters['kinematics']}" />
@@ -62,35 +62,35 @@
     <xacro:property name="wrist_3_velocity_limit" value="${sec_limits['wrist_3_joint']['max_velocity']}" scope="parent"/>
     <xacro:property name="wrist_3_effort_limit" value="${sec_limits['wrist_3_joint']['max_effort']}" scope="parent"/>
-    <!-- MOTOR DYNAMICS PARAMETERS -->
-    <xacro:property name="shoulder_pan_joint_static_friction" value="${sec_motor_dynamics['shoulder_pan_joint']['static_friction']}" scope="parent"/>
-    <xacro:property name="shoulder_pan_joint_viscous_friction" value="${sec_motor_dynamics['shoulder_pan_joint']['viscous_friction']}" scope="parent"/>
-    <xacro:property name="shoulder_pan_joint_gear_ratio" value="${sec_motor_dynamics['shoulder_pan_joint']['gear_ratio']}" scope="parent"/>
-    <xacro:property name="shoulder_pan_joint_rotor_inertia" value="${sec_motor_dynamics['shoulder_pan_joint']['rotor_inertia']}" scope="parent"/>
-    <xacro:property name="shoulder_pan_joint_reducer_inertia" value="${sec_motor_dynamics['shoulder_pan_joint']['reducer_inertia']}" scope="parent"/>
-    <xacro:property name="shoulder_lift_joint_static_friction" value="${sec_motor_dynamics['shoulder_lift_joint']['static_friction']}" scope="parent"/>
-    <xacro:property name="shoulder_lift_joint_viscous_friction" value="${sec_motor_dynamics['shoulder_lift_joint']['viscous_friction']}" scope="parent"/>
-    <xacro:property name="shoulder_lift_joint_gear_ratio" value="${sec_motor_dynamics['shoulder_lift_joint']['gear_ratio']}" scope="parent"/>
-    <xacro:property name="shoulder_lift_joint_rotor_inertia" value="${sec_motor_dynamics['shoulder_lift_joint']['rotor_inertia']}" scope="parent"/>
-    <xacro:property name="shoulder_lift_joint_reducer_inertia" value="${sec_motor_dynamics['shoulder_lift_joint']['reducer_inertia']}" scope="parent"/>
-    <xacro:property name="elbow_joint_static_friction" value="${sec_motor_dynamics['elbow_joint']['static_friction']}" scope="parent"/>
-    <xacro:property name="elbow_joint_viscous_friction" value="${sec_motor_dynamics['elbow_joint']['viscous_friction']}" scope="parent"/>
-    <xacro:property name="elbow_joint_gear_ratio" value="${sec_motor_dynamics['elbow_joint']['gear_ratio']}" scope="parent"/>
-    <xacro:property name="elbow_joint_rotor_inertia" value="${sec_motor_dynamics['elbow_joint']['rotor_inertia']}" scope="parent"/>
-    <xacro:property name="elbow_joint_reducer_inertia" value="${sec_motor_dynamics['elbow_joint']['reducer_inertia']}" scope="parent"/>
-    <xacro:property name="wrist_1_joint_static_friction" value="${sec_motor_dynamics['wrist_1_joint']['static_friction']}" scope="parent"/>
-    <xacro:property name="wrist_1_joint_viscous_friction" value="${sec_motor_dynamics['wrist_1_joint']['viscous_friction']}" scope="parent"/>
-    <xacro:property name="wrist_1_joint_gear_ratio" value="${sec_motor_dynamics['wrist_1_joint']['gear_ratio']}" scope="parent"/>
-    <xacro:property name="wrist_1_joint_rotor_inertia" value="${sec_motor_dynamics['wrist_1_joint']['rotor_inertia']}" scope="parent"/>
-    <xacro:property name="wrist_1_joint_reducer_inertia" value="${sec_motor_dynamics['wrist_1_joint']['reducer_inertia']}" scope="parent"/>
-    <xacro:property name="wrist_2_joint_static_friction" value="${sec_motor_dynamics['wrist_2_joint']['static_friction']}" scope="parent"/>
-    <xacro:property name="wrist_2_joint_viscous_friction" value="${sec_motor_dynamics['wrist_2_joint']['viscous_friction']}" scope="parent"/>
-    <xacro:property name="wrist_2_joint_gear_ratio" value="${sec_motor_dynamics['wrist_2_joint']['gear_ratio']}" scope="parent"/>
-    <xacro:property name="wrist_2_joint_rotor_inertia" value="${sec_motor_dynamics['wrist_2_joint']['rotor_inertia']}" scope="parent"/>
-    <xacro:property name="wrist_2_joint_reducer_inertia" value="${sec_motor_dynamics['wrist_2_joint']['reducer_inertia']}" scope="parent"/>
-    <xacro:property name="wrist_3_joint_static_friction" value="${sec_motor_dynamics['wrist_3_joint']['static_friction']}" scope="parent"/>
-    <xacro:property name="wrist_3_joint_viscous_friction" value="${sec_motor_dynamics['wrist_3_joint']['viscous_friction']}" scope="parent"/>
-    <xacro:property name="wrist_3_joint_gear_ratio" value="${sec_motor_dynamics['wrist_3_joint']['gear_ratio']}" scope="parent"/>
-    <xacro:property name="wrist_3_joint_rotor_inertia" value="${sec_motor_dynamics['wrist_3_joint']['rotor_inertia']}" scope="parent"/>
-    <xacro:property name="wrist_3_joint_reducer_inertia" value="${sec_motor_dynamics['wrist_3_joint']['reducer_inertia']}" scope="parent"/>
+    <!-- JOINT DYNAMICS PARAMETERS -->
+    <xacro:property name="shoulder_pan_joint_coulomb_friction" value="${sec_joint_dynamics['shoulder_pan_joint']['coulomb_friction']}" scope="parent"/>
+    <xacro:property name="shoulder_pan_joint_viscous_damping" value="${sec_joint_dynamics['shoulder_pan_joint']['viscous_damping']}" scope="parent"/>
+    <xacro:property name="shoulder_pan_joint_gear_ratio" value="${sec_joint_dynamics['shoulder_pan_joint']['gear_ratio']}" scope="parent"/>
+    <xacro:property name="shoulder_pan_joint_rotor_inertia" value="${sec_joint_dynamics['shoulder_pan_joint']['rotor_inertia']}" scope="parent"/>
+    <xacro:property name="shoulder_pan_joint_reducer_inertia" value="${sec_joint_dynamics['shoulder_pan_joint']['reducer_inertia']}" scope="parent"/>
+    <xacro:property name="shoulder_lift_joint_coulomb_friction" value="${sec_joint_dynamics['shoulder_lift_joint']['coulomb_friction']}" scope="parent"/>
+    <xacro:property name="shoulder_lift_joint_viscous_damping" value="${sec_joint_dynamics['shoulder_lift_joint']['viscous_damping']}" scope="parent"/>
+    <xacro:property name="shoulder_lift_joint_gear_ratio" value="${sec_joint_dynamics['shoulder_lift_joint']['gear_ratio']}" scope="parent"/>
+    <xacro:property name="shoulder_lift_joint_rotor_inertia" value="${sec_joint_dynamics['shoulder_lift_joint']['rotor_inertia']}" scope="parent"/>
+    <xacro:property name="shoulder_lift_joint_reducer_inertia" value="${sec_joint_dynamics['shoulder_lift_joint']['reducer_inertia']}" scope="parent"/>
+    <xacro:property name="elbow_joint_coulomb_friction" value="${sec_joint_dynamics['elbow_joint']['coulomb_friction']}" scope="parent"/>
+    <xacro:property name="elbow_joint_viscous_damping" value="${sec_joint_dynamics['elbow_joint']['viscous_damping']}" scope="parent"/>
+    <xacro:property name="elbow_joint_gear_ratio" value="${sec_joint_dynamics['elbow_joint']['gear_ratio']}" scope="parent"/>
+    <xacro:property name="elbow_joint_rotor_inertia" value="${sec_joint_dynamics['elbow_joint']['rotor_inertia']}" scope="parent"/>
+    <xacro:property name="elbow_joint_reducer_inertia" value="${sec_joint_dynamics['elbow_joint']['reducer_inertia']}" scope="parent"/>
+    <xacro:property name="wrist_1_joint_coulomb_friction" value="${sec_joint_dynamics['wrist_1_joint']['coulomb_friction']}" scope="parent"/>
+    <xacro:property name="wrist_1_joint_viscous_damping" value="${sec_joint_dynamics['wrist_1_joint']['viscous_damping']}" scope="parent"/>
+    <xacro:property name="wrist_1_joint_gear_ratio" value="${sec_joint_dynamics['wrist_1_joint']['gear_ratio']}" scope="parent"/>
+    <xacro:property name="wrist_1_joint_rotor_inertia" value="${sec_joint_dynamics['wrist_1_joint']['rotor_inertia']}" scope="parent"/>
+    <xacro:property name="wrist_1_joint_reducer_inertia" value="${sec_joint_dynamics['wrist_1_joint']['reducer_inertia']}" scope="parent"/>
+    <xacro:property name="wrist_2_joint_coulomb_friction" value="${sec_joint_dynamics['wrist_2_joint']['coulomb_friction']}" scope="parent"/>
+    <xacro:property name="wrist_2_joint_viscous_damping" value="${sec_joint_dynamics['wrist_2_joint']['viscous_damping']}" scope="parent"/>
+    <xacro:property name="wrist_2_joint_gear_ratio" value="${sec_joint_dynamics['wrist_2_joint']['gear_ratio']}" scope="parent"/>
+    <xacro:property name="wrist_2_joint_rotor_inertia" value="${sec_joint_dynamics['wrist_2_joint']['rotor_inertia']}" scope="parent"/>
+    <xacro:property name="wrist_2_joint_reducer_inertia" value="${sec_joint_dynamics['wrist_2_joint']['reducer_inertia']}" scope="parent"/>
+    <xacro:property name="wrist_3_joint_coulomb_friction" value="${sec_joint_dynamics['wrist_3_joint']['coulomb_friction']}" scope="parent"/>
+    <xacro:property name="wrist_3_joint_viscous_damping" value="${sec_joint_dynamics['wrist_3_joint']['viscous_damping']}" scope="parent"/>
+    <xacro:property name="wrist_3_joint_gear_ratio" value="${sec_joint_dynamics['wrist_3_joint']['gear_ratio']}" scope="parent"/>
+    <xacro:property name="wrist_3_joint_rotor_inertia" value="${sec_joint_dynamics['wrist_3_joint']['rotor_inertia']}" scope="parent"/>
+    <xacro:property name="wrist_3_joint_reducer_inertia" value="${sec_joint_dynamics['wrist_3_joint']['reducer_inertia']}" scope="parent"/>
     <!-- kinematics -->
     <xacro:property name="shoulder_x" value="${sec_kinematics['shoulder']['x']}" scope="parent"/>

File: ur_description/urdf/inc/ur_macro.xacro (robot description, xacro)
@@ -281,9 +281,13 @@
       </xacro:if>
       <dynamics damping="0" friction="0"/>
-      <motor_dynamics static_friction="${shoulder_pan_joint_static_friction}"
-                      viscous_friction="${shoulder_pan_joint_viscous_friction}"
-                      gear_ratio="${shoulder_pan_joint_gear_ratio}"
-                      rotor_inertia="${shoulder_pan_joint_rotor_inertia}"
-                      reducer_inertia="${shoulder_pan_joint_reducer_inertia}"/>
+      <!--
+        NB: We use `chef_dynamics` instead of `dynamics` when doing joint-torque calculations in planning;
+        `dynamics` does not have all the params we need to properly model the joint for calculating torque.
+      -->
+      <chef_dynamics coulomb_friction="${shoulder_pan_joint_coulomb_friction}"
+                     viscous_damping="${shoulder_pan_joint_viscous_damping}"
+                     gear_ratio="${shoulder_pan_joint_gear_ratio}"
+                     rotor_inertia="${shoulder_pan_joint_rotor_inertia}"
+                     reducer_inertia="${shoulder_pan_joint_reducer_inertia}"/>
     </joint>
     <joint name="${prefix}shoulder_lift_joint" type="revolute">
@@ -298,9 +302,9 @@
       </xacro:if>
       <dynamics damping="0" friction="0"/>
-      <motor_dynamics static_friction="${shoulder_lift_joint_static_friction}"
-                      viscous_friction="${shoulder_lift_joint_viscous_friction}"
-                      gear_ratio="${shoulder_lift_joint_gear_ratio}"
-                      rotor_inertia="${shoulder_lift_joint_rotor_inertia}"
-                      reducer_inertia="${shoulder_lift_joint_reducer_inertia}"/>
+      <chef_dynamics coulomb_friction="${shoulder_lift_joint_coulomb_friction}"
+                     viscous_damping="${shoulder_lift_joint_viscous_damping}"
+                     gear_ratio="${shoulder_lift_joint_gear_ratio}"
+                     rotor_inertia="${shoulder_lift_joint_rotor_inertia}"
+                     reducer_inertia="${shoulder_lift_joint_reducer_inertia}"/>
     </joint>
     <joint name="${prefix}elbow_joint" type="revolute">
@@ -315,9 +319,9 @@
       </xacro:if>
       <dynamics damping="0" friction="0"/>
-      <motor_dynamics static_friction="${elbow_joint_static_friction}"
-                      viscous_friction="${elbow_joint_viscous_friction}"
-                      gear_ratio="${elbow_joint_gear_ratio}"
-                      rotor_inertia="${elbow_joint_rotor_inertia}"
-                      reducer_inertia="${elbow_joint_reducer_inertia}"/>
+      <chef_dynamics coulomb_friction="${elbow_joint_coulomb_friction}"
+                     viscous_damping="${elbow_joint_viscous_damping}"
+                     gear_ratio="${elbow_joint_gear_ratio}"
+                     rotor_inertia="${elbow_joint_rotor_inertia}"
+                     reducer_inertia="${elbow_joint_reducer_inertia}"/>
     </joint>
     <joint name="${prefix}wrist_1_joint" type="revolute">
@@ -332,9 +336,9 @@
       </xacro:if>
       <dynamics damping="0" friction="0"/>
-      <motor_dynamics static_friction="${wrist_1_joint_static_friction}"
-                      viscous_friction="${wrist_1_joint_viscous_friction}"
-                      gear_ratio="${wrist_1_joint_gear_ratio}"
-                      rotor_inertia="${wrist_1_joint_rotor_inertia}"
-                      reducer_inertia="${wrist_1_joint_reducer_inertia}"/>
+      <chef_dynamics coulomb_friction="${wrist_1_joint_coulomb_friction}"
+                     viscous_damping="${wrist_1_joint_viscous_damping}"
+                     gear_ratio="${wrist_1_joint_gear_ratio}"
+                     rotor_inertia="${wrist_1_joint_rotor_inertia}"
+                     reducer_inertia="${wrist_1_joint_reducer_inertia}"/>
     </joint>
     <joint name="${prefix}wrist_2_joint" type="revolute">
@@ -349,9 +353,9 @@
       </xacro:if>
       <dynamics damping="0" friction="0"/>
-      <motor_dynamics static_friction="${wrist_2_joint_static_friction}"
-                      viscous_friction="${wrist_2_joint_viscous_friction}"
-                      gear_ratio="${wrist_2_joint_gear_ratio}"
-                      rotor_inertia="${wrist_2_joint_rotor_inertia}"
-                      reducer_inertia="${wrist_2_joint_reducer_inertia}"/>
+      <chef_dynamics coulomb_friction="${wrist_2_joint_coulomb_friction}"
+                     viscous_damping="${wrist_2_joint_viscous_damping}"
+                     gear_ratio="${wrist_2_joint_gear_ratio}"
+                     rotor_inertia="${wrist_2_joint_rotor_inertia}"
+                     reducer_inertia="${wrist_2_joint_reducer_inertia}"/>
     </joint>
     <joint name="${prefix}wrist_3_joint" type="revolute">
@@ -366,9 +370,9 @@
       </xacro:if>
       <dynamics damping="0" friction="0"/>
-      <motor_dynamics static_friction="${wrist_3_joint_static_friction}"
-                      viscous_friction="${wrist_3_joint_viscous_friction}"
-                      gear_ratio="${wrist_3_joint_gear_ratio}"
-                      rotor_inertia="${wrist_3_joint_rotor_inertia}"
-                      reducer_inertia="${wrist_3_joint_reducer_inertia}"/>
+      <chef_dynamics coulomb_friction="${wrist_3_joint_coulomb_friction}"
+                     viscous_damping="${wrist_3_joint_viscous_damping}"
+                     gear_ratio="${wrist_3_joint_gear_ratio}"
+                     rotor_inertia="${wrist_3_joint_rotor_inertia}"
+                     reducer_inertia="${wrist_3_joint_reducer_inertia}"/>
     </joint>
     <!-- ROS-Industrial 'base' frame: base_link to UR 'Base' Coordinates transform -->
